File: MCU.sch (KiCad schematic (older format))
At the start: 14 parts, among them U7 STM32F405RGTx, U8 ADR4533BRZ, Y1 Crystal_GND24

Commit message: almost done with bom. there are some issues
Parts:
- C20, C21: value 22p -> 15p; OrderN (none) -> 311-1060-1-ND
- C22, C23, C24, C25, C26, C27, C29, C30, C5: OrderN (none) -> 490-10731-1-ND
- U7: OrderN (none) -> 497-11767-ND
- Y1: OrderN (none) -> 535-9720-1-ND
Changed lines of the file:
@@
 F 2 "Package_QFP:LQFP-64_10x10mm_P0.5mm" H 5150 1900 50  0001 R CNN
 F 3 "http://www.st.com/st-web-ui/static/active/en/resource/technical/document/datasheet/DM00037051.pdf" H 5750 3600 50  0001 C CNN
+F 4 "497-11767-ND" H 5750 3600 50  0001 C CNN "OrderN"
 	1    5750 3600
 	1    0    0    -1
@@
 F 2 "Capacitor_SMD:C_0603_1608Metric" H 4750 2350 50  0001 C CNN
 F 3 "~" H 4750 2350 50  0001 C CNN
+F 4 "490-10731-1-ND" H 4750 2350 50  0001 C CNN "OrderN"
 	1    4750 2350
 	0    1    1    0
@@
 F 2 "Capacitor_SMD:C_0603_1608Metric" H 4750 2550 50  0001 C CNN
 F 3 "~" H 4750 2550 50  0001 C CNN
+F 4 "490-10731-1-ND" H 4750 2550 50  0001 C CNN "OrderN"
 	1    4750 2550
 	0    1    1    0
@@
 P 3350 2850
 F 0 "C20" H 3442 2896 50  0000 L CNN
-F 1 "22p" H 3442 2805 50  0000 L CNN
+F 1 "15p" H 3442 2805 50  0000 L CNN
 F 2 "Capacitor_SMD:C_0603_1608Metric" H 3350 2850 50  0001 C CNN
 F 3 "~" H 3350 2850 50  0001 C CNN
+F 4 "311-1060-1-ND" H 3350 2850 50  0001 C CNN "OrderN"
 	1    3350 2850
 	1    0    0    -1
@@
 P 3350 3450
 F 0 "C21" H 3442 3496 50  0000 L CNN
-F 1 "22p" H 3442 3405 50  0000 L CNN
+F 1 "15p" H 3442 3405 50  0000 L CNN
 F 2 "Capacitor_SMD:C_0603_1608Metric" H 3350 3450 50  0001 C CNN
 F 3 "~" H 3350 3450 50  0001 C CNN
+F 4 "311-1060-1-ND" H 3350 3450 50  0001 C CNN "OrderN"
 	1    3350 3450
 	1    0    0    -1
@@
 F 2 "Crystal:Crystal_SMD_Abracon_ABM3C-4Pin_5.0x3.2mm" H 3900 3250 50  0001 C CNN
 F 3 "~" H 3900 3250 50  0001 C CNN
+F 4 "535-9720-1-ND" H 3900 3250 50  0001 C CNN "OrderN"
 	1    3900 3250
 	0    1    1    0
@@
 F 2 "Capacitor_SMD:C_0603_1608Metric" H 4800 1400 50  0001 C CNN
 F 3 "~" H 4800 1400 50  0001 C CNN
+F 4 "490-10731-1-ND" H 4800 1400 50  0001 C CNN "OrderN"
 	1    4800 1400
 	-1   0    0    1
@@
 F 2 "Capacitor_SMD:C_0603_1608Metric" H 4600 1400 50  0001 C CNN
 F 3 "~" H 4600 1400 50  0001 C CNN
+F 4 "490-10731-1-ND" H 4600 1400 50  0001 C CNN "OrderN"
 	1    4600 1400
 	-1   0    0    1
@@
 F 2 "Capacitor_SMD:C_0603_1608Metric" H 4400 1400 50  0001 C CNN
 F 3 "~" H 4400 1400 50  0001 C CNN
+F 4 "490-10731-1-ND" H 4400 1400 50  0001 C CNN "OrderN"
 	1    4400 1400
 	-1   0    0    1
@@
 F 2 "Capacitor_SMD:C_0603_1608Metric" H 4200 1400 50  0001 C CNN
 F 3 "~" H 4200 1400 50  0001 C CNN
+F 4 "490-10731-1-ND" H 4200 1400 50  0001 C CNN "OrderN"
 	1    4200 1400
 	-1   0    0    1
@@
 F 2 "Capacitor_SMD:C_0603_1608Metric" H 6750 1350 50  0001 C CNN
 F 3 "~" H 6750 1350 50  0001 C CNN
+F 4 "490-10731-1-ND" H 6750 1350 50  0001 C CNN "OrderN"
 	1    6750 1350
 	-1   0    0    1
@@
 F 2 "Capacitor_SMD:C_0603_1608Metric" H 7350 1450 50  0001 C CNN
 F 3 "~" H 7350 1450 50  0001 C CNN
+F 4 "490-10731-1-ND" H 7350 1450 50  0001 C CNN "OrderN"
 	1    7350 1450
 	-1   0    0    1
@@
 F 2 "Capacitor_SMD:C_0603_1608Metric" H 5000 1400 50  0001 C CNN
 F 3 "~" H 5000 1400 50  0001 C CNN
+F 4 "490-10731-1-ND" H 5000 1400 50  0001 C CNN "OrderN"
 	1    5000 1400
 	-1   0    0    1
