File: power.sch (KiCad schematic (older format))
At the start: 17 parts, among them U10 AZ1117-3.3, U9 TPS54160

Commit message: almost done with bom. there are some issues
Parts:
- C31, C33, C36, C37: OrderN (none) -> 445-5207-1-ND
- C32, C39: OrderN (none) -> 399-1089-1-ND
- C34: OrderN (none) -> 1276-1160-1-ND
- C35: value 100n -> 0.1u; OrderN (none) -> 1276-1000-1-ND
- C38: OrderN (none) -> 493-11709-1-ND
- R31: OrderN (none) -> 311-220KHRCT-ND
- R32: OrderN (none) -> 311-15.0KHRCT-ND
- R33: OrderN (none) -> 311-18.0KHRCT-ND
- R34: OrderN (none) -> 311-3.30KHRCT-ND
Changed lines of the file:
@@
 P 5850 2300
 F 0 "C35" V 5800 2450 50  0000 C CNN
-F 1 "100n" V 5712 2300 50  0000 C CNN
+F 1 "0.1u" V 5712 2300 50  0000 C CNN
 F 2 "Capacitor_SMD:C_0603_1608Metric" H 5850 2300 50  0001 C CNN
 F 3 "~" H 5850 2300 50  0001 C CNN
+F 4 "1276-1000-1-ND" H 5850 2300 50  0001 C CNN "OrderN"
 	1    5850 2300
 	0    1    1    0
@@
 F 2 "Resistor_SMD:R_0603_1608Metric" H 6800 3100 50  0001 C CNN
 F 3 "~" H 6800 3100 50  0001 C CNN
+F 4 " 311-3.30KHRCT-ND" H 6800 3100 50  0001 C CNN "OrderN"
 	1    6800 3100
 	-1   0    0    1
@@
 F 2 "Resistor_SMD:R_0603_1608Metric" H 6800 2650 50  0001 C CNN
 F 3 "~" H 6800 2650 50  0001 C CNN
+F 4 "311-18.0KHRCT-ND " H 6800 2650 50  0001 C CNN "OrderN"
 	1    6800 2650
 	1    0    0    -1
@@
 F 2 "Capacitor_SMD:C_1206_3216Metric" H 3450 2450 50  0001 C CNN
 F 3 "~" H 3450 2450 50  0001 C CNN
+F 4 "445-5207-1-ND" H 3450 2450 50  0001 C CNN "OrderN"
 	1    3450 2450
 	1    0    0    -1
@@
 F 2 "Resistor_SMD:R_0603_1608Metric" H 3950 3050 50  0001 C CNN
 F 3 "~" H 3950 3050 50  0001 C CNN
+F 4 "311-220KHRCT-ND" H 3950 3050 50  0001 C CNN "OrderN"
 	1    3950 3050
 	1    0    0    -1
@@
 F 2 "Resistor_SMD:R_0603_1608Metric" H 4200 3050 50  0001 C CNN
 F 3 "~" H 4200 3050 50  0001 C CNN
+F 4 "311-15.0KHRCT-ND" H 4200 3050 50  0001 C CNN "OrderN"
 	1    4200 3050
 	1    0    0    -1
@@
 F 2 "Capacitor_SMD:C_0603_1608Metric" H 4200 3400 50  0001 C CNN
 F 3 "~" H 4200 3400 50  0001 C CNN
+F 4 " 399-1089-1-ND " H 4200 3400 50  0001 C CNN "OrderN"
 	1    4200 3400
 	-1   0    0    1
@@
 F 2 "Capacitor_SMD:C_0603_1608Metric" H 4450 3250 50  0001 C CNN
 F 3 "~" H 4450 3250 50  0001 C CNN
+F 4 "1276-1160-1-ND " H 4450 3250 50  0001 C CNN "OrderN"
 	1    4450 3250
 	-1   0    0    1
@@
 F 2 "Capacitor_SMD:C_1206_3216Metric" H 7250 3000 50  0001 C CNN
 F 3 "~" H 7250 3000 50  0001 C CNN
+F 4 "445-5207-1-ND" H 7250 3000 50  0001 C CNN "OrderN"
 	1    7250 3000
 	1    0    0    -1
@@
 F 3 "~" H 7650 3000 50  0001 C CNN
 F 4 "https://www.digikey.se/product-detail/en/nichicon/URS1C471MPD1TD/493-11709-1-ND/4320195" H 7650 3000 50  0001 C CNN "digikey"
+F 5 "493-11709-1-ND" H 7650 3000 50  0001 C CNN "OrderN"
 	1    7650 3000
 	1    0    0    -1
@@
 F 2 "Capacitor_SMD:C_1206_3216Metric" H 4350 5000 50  0001 C CNN
 F 3 "~" H 4350 5000 50  0001 C CNN
+F 4 "445-5207-1-ND" H 4350 5000 50  0001 C CNN "OrderN"
 	1    4350 5000
 	1    0    0    -1
@@
 F 2 "Capacitor_SMD:C_1206_3216Metric" H 5900 5000 50  0001 C CNN
 F 3 "~" H 5900 5000 50  0001 C CNN
+F 4 "445-5207-1-ND" H 5900 5000 50  0001 C CNN "OrderN"
 	1    5900 5000
 	1    0    0    -1
@@
 F 2 "Capacitor_SMD:C_0603_1608Metric" H 3650 3400 50  0001 C CNN
 F 3 "~" H 3650 3400 50  0001 C CNN
+F 4 " 399-1089-1-ND " H 3650 3400 50  0001 C CNN "OrderN"
 	1    3650 3400
 	-1   0    0    1
