File: output.sch (KiCad schematic (older format))
At the start: 16 parts, among them U1 OPA549, U2 INA240A1PW, U3 OPA549, U4 INA240A1PW

Commit message: Added testpoints, changed connectors, changed shunts
Parts:
- R14, R17: footprint Resistor_SMD:R_Shunt_Ohmite_LVK12 -> Resistor_SMD:R_Shunt_Ohmite_LVK24; OrderN LVK12R010DERCT-ND -> LVK24R010DERCT-ND
Changed lines of the file:
@@
 F 0 "R17" V 9185 2700 50  0000 C CNN
 F 1 "r_shunt_lvk" V 9276 2700 50  0000 C CNN
-F 2 "Resistor_SMD:R_Shunt_Ohmite_LVK12" H 9400 2700 50  0001 C CNN
+F 2 "Resistor_SMD:R_Shunt_Ohmite_LVK24" H 9400 2700 50  0001 C CNN
 F 3 "" H 9400 2700 50  0001 C CNN
-F 4 "LVK12R010DERCT-ND" V 9400 2700 50  0001 C CNN "OrderN"
+F 4 "LVK24R010DERCT-ND" V 9400 2700 50  0001 C CNN "OrderN"
 	1    9400 2700
 	0    1    1    0
@@
 F 0 "R14" V 3535 3200 50  0000 C CNN
 F 1 "r_shunt_lvk" V 3626 3200 50  0000 C CNN
-F 2 "Resistor_SMD:R_Shunt_Ohmite_LVK12" H 3750 3200 50  0001 C CNN
+F 2 "Resistor_SMD:R_Shunt_Ohmite_LVK24" H 3750 3200 50  0001 C CNN
 F 3 "" H 3750 3200 50  0001 C CNN
-F 4 "LVK12R010DERCT-ND" V 3750 3200 50  0001 C CNN "OrderN"
+F 4 "LVK24R010DERCT-ND" V 3750 3200 50  0001 C CNN "OrderN"
 	1    3750 3200
 	0    1    1    0

Commit message: all components now have an OrderN in the matrix
Parts:
- U2, U4: OrderN (none) -> 296-45088-2-ND
Changed lines of the file:
@@
 F 2 "Package_SO:TSSOP-8_4.4x3mm_P0.65mm" H 3750 3250 50  0001 C CNN
 F 3 "http://www.ti.com/lit/ds/symlink/ina240.pdf" H 3900 4050 50  0001 C CNN
+F 4 " 296-45088-2-ND" H 3750 3900 50  0001 C CNN "OrderN"
 	1    3750 3900
 	0    1    1    0
@@
 F 2 "Package_SO:TSSOP-8_4.4x3mm_P0.65mm" H 9400 2750 50  0001 C CNN
 F 3 "http://www.ti.com/lit/ds/symlink/ina240.pdf" H 9550 3550 50  0001 C CNN
+F 4 " 296-45088-2-ND" H 9400 3400 50  0001 C CNN "OrderN"
 	1    9400 3400
 	0    1    1    0
